File: PCB/bpod_stepper_1.1.sch (EAGLE design)
At the start: 26 parts, among them IC1 LM3480-5.0, IC2 SN65HVD31DR, J1 282841-4, J8 POWER_JACK

Commit message: corrected wrong routing for RX & TX
Connections:
- net RX1: now also IC2.R; no longer IC2.D
- net TX1: now also IC2.D; no longer IC2.R
Changed lines of the file:
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@@
 </segment>
 <segment>
-<pinref part="IC2" gate="G$1" pin="R"/>
-<wire x1="71.12" y1="83.82" x2="63.5" y2="83.82" width="0.1524" layer="91"/>
-<label x="73.66" y="83.82" size="1.778" layer="95"/>
+<pinref part="IC2" gate="G$1" pin="D"/>
+<wire x1="63.5" y1="86.36" x2="73.66" y2="86.36" width="0.1524" layer="91"/>
+<label x="73.66" y="86.36" size="1.778" layer="95"/>
 </segment>
 </net>
@@
 </segment>
 <segment>
-<pinref part="IC2" gate="G$1" pin="D"/>
-<wire x1="63.5" y1="86.36" x2="68.58" y2="86.36" width="0.1524" layer="91"/>
-<label x="73.66" y="86.36" size="1.778" layer="95"/>
+<pinref part="IC2" gate="G$1" pin="R"/>
+<wire x1="63.5" y1="83.82" x2="73.66" y2="83.82" width="0.1524" layer="91"/>
+<label x="73.66" y="83.82" size="1.778" layer="95"/>
 </segment>
 </net>
