File: PCB/bpod_stepper_1.5.4.brd (EAGLE design)
At the start: 83.8 x 66 mm, 36 parts, among them IC1 MCP1792T-5002H/DB, IC2 SN65HVD31DR, IC3 MCP1792T-5002H/DB, IC4 MCP1793, J8 POWER_JACK

Commit message: some clean-up, undo version increment
Parts:
- moved C10 7.74 mm to (9.14, 42.7), turned to 270 degrees
- moved C4 2.17 mm to (47.8, 17.5), turned to 0 degrees
- moved C9 0.72 mm to (13.7, 42.7), turned to 270 degrees
- moved C3 0.57 mm to (45.7, 9.65)
Connections:
- net GND: no longer TEENSY.23/A9
Routing:
- net VMOTOR: track 119.9 -> 117.4 mm
- net BOOL_VM: track 59.0 -> 58.0 mm
Changed lines of the file:
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@@
 <layer number="25" name="tNames" color="7" fill="1" visible="yes" active="yes"/>
 <layer number="26" name="bNames" color="7" fill="1" visible="yes" active="yes"/>
-<layer number="27" name="tValues" color="7" fill="1" visible="no" active="yes"/>
+<layer number="27" name="tValues" color="7" fill="1" visible="yes" active="yes"/>
 <layer number="28" name="bValues" color="7" fill="1" visible="no" active="yes"/>
 <layer number="29" name="tStop" color="7" fill="3" visible="no" active="yes"/>
@@
 </element>
 <element name="IC4" library="MCP1793" package="SOT223-5" value="MCP1793" x="51.435" y="12.7" smashed="yes" rot="R270">
-<attribute name="NAME" x="51.435" y="16.51" size="0.8128" layer="25" font="vector" align="bottom-center"/>
+<attribute name="NAME" x="51.435" y="8.89" size="0.8128" layer="25" font="vector" align="top-center"/>
 <attribute name="VALUE" x="51.2445" y="12.7" size="0.4064" layer="27" font="vector" rot="R270" align="bottom-center"/>
 </element>
 <element name="D12" library="we-rcl" package="SOD123" value="S310FA" x="44.45" y="13.97" smashed="yes" rot="R270">
-<attribute name="NAME" x="43.18" y="15.875" size="0.8128" layer="25" font="vector" rot="R180" align="center"/>
+<attribute name="NAME" x="44.45" y="15.621" size="0.8128" layer="25" font="vector" rot="R180" align="center"/>
 </element>
 <element name="IC3" library="MCP1792_3" package="SOT223" value="MCP1792T-5002H/DB" x="11.43" y="49.8475" smashed="yes">
-<attribute name="NAME" x="8.382" y="44.6405" size="0.8128" layer="25" font="vector" align="top-left"/>
+<attribute name="NAME" x="13.716" y="52.832" size="0.8128" layer="25" font="vector" align="top-left"/>
 <attribute name="VALUE" x="10.3505" y="49.657" size="0.4064" layer="27"/>
 </element>
@@
 <attribute name="VALUE" x="49.0855" y="60.5155" size="0.4064" layer="27" rot="R90"/>
 </element>
-<element name="C3" library="SparkFun-Capacitors" package="1206@1" value="2.2uf" x="45.212" y="9.398" smashed="yes" rot="R270">
-<attribute name="NAME" x="43.053" y="9.906" size="0.8128" layer="25" font="vector" rot="R270"/>
-<attribute name="VALUE" x="43.688" y="10.795" size="0.4064" layer="27" rot="R270"/>
-</element>
-<element name="C4" library="SparkFun-Capacitors" package="1206@1" value="2.2uf" x="45.72" y="18.288" smashed="yes" rot="R90">
-<attribute name="NAME" x="46.228" y="21.971" size="0.8128" layer="25" font="vector" rot="R180"/>
-<attribute name="VALUE" x="47.244" y="16.891" size="0.4064" layer="27" rot="R90"/>
-</element>
-<element name="C9" library="SparkFun-Capacitors" package="1206@1" value="1uf" x="13.208" y="43.18" smashed="yes" rot="R180">
-<attribute name="NAME" x="13.716" y="41.529" size="0.8128" layer="25" font="vector" rot="R180"/>
-<attribute name="VALUE" x="14.605" y="44.704" size="0.4064" layer="27" rot="R180"/>
-</element>
-<element name="C10" library="SparkFun-Capacitors" package="1206@1" value="1uf" x="6.096" y="49.784" smashed="yes" rot="R90">
-<attribute name="NAME" x="7.112" y="53.467" size="0.8128" layer="25" font="vector" rot="R180"/>
-<attribute name="VALUE" x="7.62" y="48.387" size="0.4064" layer="27" rot="R90"/>
+<element name="C3" library="SparkFun-Capacitors" package="1206@1" value="2.2uf" x="45.72" y="9.652" smashed="yes" rot="R270">
+<attribute name="NAME" x="44.323" y="9.652" size="0.8128" layer="25" font="vector" align="center-right"/>
+</element>
+<element name="C4" library="SparkFun-Capacitors" package="1206@1" value="2.2uf" x="47.752" y="17.526" smashed="yes">
+<attribute name="NAME" x="47.752" y="18.923" size="0.8128" layer="25" font="vector" align="bottom-center"/>
+</element>
+<element name="C9" library="SparkFun-Capacitors" package="1206@1" value="1uf" x="13.716" y="42.672" smashed="yes" rot="R270">
+<attribute name="NAME" x="13.716" y="39.878" size="0.8128" layer="25" font="vector" align="top-center"/>
+</element>
+<element name="C10" library="SparkFun-Capacitors" package="1206@1" value="1uf" x="9.144" y="42.672" smashed="yes" rot="R270">
+<attribute name="NAME" x="9.144" y="39.878" size="0.8128" layer="25" font="vector" align="top-center"/>
 </element>
 </elements>
@@
 <contactref element="C9" pad="2"/>
 <contactref element="C10" pad="2"/>
-<contactref element="TEENSY" pad="23/A9"/>
 </signal>
 <signal name="TX1">
@@
 <wire x1="16.51" y1="56.2" x2="17.34" y2="54.8755" width="1.27" layer="1"/>
 <wire x1="17.34" y1="54.8755" x2="17.34" y2="49.8475" width="1.27" layer="1"/>
-<wire x1="17.34" y1="49.8475" x2="17.34" y2="49.60586875" width="1.27" layer="1"/>
 <wire x1="16.51" y1="56.2" x2="16.51" y2="57.14" width="1.27" layer="1"/>
 <wire x1="16.51" y1="57.14" x2="25.0825" y2="57.14" width="1.27" layer="1"/>
@@
 <contactref element="IC3" pad="1"/>
 <contactref element="C10" pad="1"/>
-<wire x1="8.33386875" y1="49.60586875" x2="7.112" y2="48.384" width="1.016" layer="1"/>
-<wire x1="7.112" y1="48.384" x2="6.096" y2="48.384" width="1.016" layer="1"/>
-<wire x1="17.34" y1="49.60586875" x2="8.33386875" y2="49.60586875" width="1.016" layer="1"/>
-<wire x1="6.096" y1="48.384" x2="7.7313" y2="46.7487" width="1.016" layer="1"/>
-<wire x1="7.7313" y1="46.7487" x2="9.1186" y2="46.7487" width="1.016" layer="1"/>
+<wire x1="10.414" y1="49.8475" x2="17.34" y2="49.8475" width="1.016" layer="1"/>
+<wire x1="9.1186" y1="46.7487" x2="9.1186" y2="44.0974" width="0.762" layer="1"/>
+<wire x1="9.1186" y1="44.0974" x2="9.144" y2="44.072" width="0.762" layer="1"/>
+<wire x1="9.1186" y1="46.7487" x2="9.1186" y2="48.5521" width="1.016" layer="1"/>
+<wire x1="9.1186" y1="48.5521" x2="10.414" y2="49.8475" width="1.016" layer="1"/>
 </signal>
 <signal name="EN">
@@
 <contactref element="C8" pad="1"/>
 <contactref element="IC4" pad="4"/>
-<wire x1="48.2346" y1="11.43" x2="46.482" y2="11.43" width="0.6096" layer="1"/>
-<wire x1="45.844" y1="11.43" x2="13.7825" y2="11.43" width="0.6096" layer="1"/>
+<wire x1="48.2346" y1="11.43" x2="46.098" y2="11.43" width="0.6096" layer="1"/>
+<wire x1="46.098" y1="11.43" x2="13.7825" y2="11.43" width="0.6096" layer="1"/>
 <wire x1="13.335" y1="11.43" x2="13.7825" y2="11.43" width="0.6096" layer="1"/>
 <wire x1="13.335" y1="17.78" x2="13.335" y2="11.43" width="0.6096" layer="1"/>
 <contactref element="C3" pad="1"/>
-<wire x1="45.212" y1="10.798" x2="45.844" y2="11.43" width="0.6096" layer="1"/>
-<wire x1="45.844" y1="11.43" x2="46.482" y2="11.43" width="0.6096" layer="1"/>
+<wire x1="45.72" y1="11.052" x2="46.098" y2="11.43" width="0.6096" layer="1"/>
 </signal>
 <signal name="VIO_CTRL">
@@
 <contactref element="D3" pad="A"/>
 <contactref element="TEENSY" pad="4"/>
-<wire x1="56.515" y1="50.8" x2="51.435" y2="45.72" width="0.762" layer="1"/>
+<wire x1="51.435" y1="45.72" x2="56.515" y2="50.8" width="0.762" layer="1"/>
 <wire x1="57.785" y1="50.8" x2="56.515" y2="50.8" width="0.762" layer="1"/>
 <wire x1="66.3575" y1="50.4875" x2="66.045" y2="50.8" width="0.762" layer="1"/>
 <wire x1="66.045" y1="50.8" x2="57.785" y2="50.8" width="0.762" layer="1"/>
-<wire x1="17.45" y1="45.72" x2="51.435" y2="45.72" width="0.762" layer="1"/>
 <contactref element="IC3" pad="3"/>
 <contactref element="C9" pad="1"/>
-<wire x1="14.608" y1="45.8821" x2="14.608" y2="43.18" width="0.762" layer="1"/>
-<wire x1="13.7414" y1="46.7487" x2="14.608" y2="45.8821" width="0.762" layer="1"/>
-<wire x1="14.608" y1="43.18" x2="14.91" y2="43.18" width="0.762" layer="1"/>
-<wire x1="14.91" y1="43.18" x2="17.45" y2="45.72" width="0.762" layer="1"/>
+<wire x1="13.7414" y1="46.7487" x2="13.7414" y2="44.0974" width="0.762" layer="1"/>
+<wire x1="13.7414" y1="44.0974" x2="13.716" y2="44.072" width="0.762" layer="1"/>
+<wire x1="16.0401" y1="45.72" x2="15.0114" y2="46.7487" width="0.762" layer="1"/>
+<wire x1="13.7414" y1="46.7487" x2="15.0114" y2="46.7487" width="0.762" layer="1"/>
+<wire x1="16.0401" y1="45.72" x2="51.435" y2="45.72" width="0.762" layer="1"/>
 </signal>
 <signal name="AGND">
@@
 <contactref element="D12" pad="C"/>
 <contactref element="IC4" pad="2"/>
-<wire x1="46.05" y1="13.97" x2="46.482" y2="13.97" width="0.6096" layer="1"/>
 <contactref element="C4" pad="1"/>
-<wire x1="46.482" y1="13.97" x2="48.2346" y2="13.97" width="0.6096" layer="1"/>
-<wire x1="45.72" y1="16.888" x2="46.482" y2="16.126" width="0.6096" layer="1"/>
-<wire x1="46.482" y1="16.126" x2="46.482" y2="13.97" width="0.6096" layer="1"/>
+<wire x1="46.05" y1="13.97" x2="48.2346" y2="13.97" width="0.6096" layer="1"/>
+<wire x1="46.352" y1="17.526" x2="46.05" y2="17.224" width="0.6096" layer="1"/>
+<wire x1="46.05" y1="13.97" x2="46.05" y2="17.224" width="0.6096" layer="1"/>
 </signal>
 </signals>
