File: PCB/bpod_stepper_1.5.4.sch (EAGLE design)
At the start: 32 parts, among them IC1 MCP1792T-5002H/DB, IC2 SN65HVD31DR, IC3 MCP1792T-5002H/DB, IC4 MCP1793, J8 POWER_JACK

Commit message: some clean-up, undo version increment
Connections:
- net GND: no longer TEENSY.23/A9/T/PWM
Changed lines of the file:
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@@
 <label x="147.32" y="110.49" size="1.778" layer="95"/>
-</segment>
-<segment>
-<pinref part="TEENSY" gate="G$1" pin="23/A9/T/PWM"/>
-<wire x1="162.56" y1="107.95" x2="147.32" y2="107.95" width="0.1524" layer="91"/>
-<label x="147.32" y="108.204" size="1.778" layer="95"/>
 </segment>
 </net>
